Commit message: ECE569 Lab2 complete Steps 1 to 4

File: Step1/r3bot.urdf (robot description, URDF)
Before this commit: robot rrbot, 5 links, 4 joints
Links:
- added link link3; visual box size=0.05 0.05 0.5
Joints:
- added joint joint3: type revolute, parent link2, child link3, origin xyz=0 0.05 0.9 rpy=0 0 0, axis 0 1 0, limit lower=-1.57 upper=1.57 effort=1 velocity=1
- joint joint1: limit (none) -> lower=-1.57 upper=1.57 effort=1 velocity=1; type continuous -> revolute
- joint joint2: limit (none) -> lower=-1.57 upper=1.57 effort=1 velocity=1; type continuous -> revolute
- joint tool_joint: origin xyz=0 0 0.95 rpy=0 0 0 -> xyz=0 0 0.45 rpy=0 0 0; parent link2 -> link3

File: Step2/rrbot_macro.xacro (robot description, xacro)
@@ -5,5 +5,5 @@
     <xacro:property name="width" value="0.05" /> <!-- Square dimensions (widthxwidth) of beams -->
     <xacro:property name="height0" value="2" /> <!-- base_link -->
-    <xacro:property name="height1" value="1" /> <!-- link1 -->
+    <xacro:property name="height1" value="1.5" /> <!-- link1 -->
     <xacro:property name="height2" value="1" /> <!-- link2 -->
     <xacro:property name="axel_offset" value="0.05" /> <!-- Space between top of beam and each joint -->

File: Step2/rrbot_on_table.urdf.xacro (robot description, xacro)
@@ -9,5 +9,5 @@
     </xacro:table>
     <xacro:rrbot prefix="rrbot_" parent="table_top">
-        <origin xyz="0 0 0" rpy="0 0 0" />
+      <origin xyz="0 0 0" rpy="0 0 0"/>
     </xacro:rrbot>
 </robot>

File: Step2/table_on_rrbot.urdf.xacro (robot description, xacro)
@@ -1,13 +1,16 @@
 <?xml version="1.0" encoding="UTF-8"?>
-<robot xmlns:xacro="http://wiki.ros.org/xacro" name="table">
-    <xacro:include filename="materials.xacro" />
-    <xacro:include filename="table_macro.xacro" />
-    <xacro:include filename="rrbot_macro.xacro" />
-    <link name="world" />
-    <xacro:rrbot prefix="rrbot_" parent="world">
-        <origin xyz="0 0 0" rpy="0 0 0" />
-    </xacro:rrbot>
-    <xacro:table prefix="table_" parent="rrbot_tool0">
-        <origin xyz="0 0 0" rpy="${pi} 0 0" />
-    </xacro:table>
+<robot xmlns:xacro="http://www.ros.org/wiki/xacro" name="table_on_rrbot">
+  <xacro:include filename="materials.xacro"/>
+  <xacro:include filename="rrbot_macro.xacro"/>
+  <xacro:include filename="table_macro.xacro"/>
+  <!-- world frame -->
+  <link name="world"/>
+  <!-- Create Robot -->
+  <xacro:rrbot prefix="rrbot_" parent="world">
+    <origin xyz="0 0 0" rpy="0 0 0"/>
+  </xacro:rrbot>
+  <!-- Mount table to END EFFECTOR -->
+  <xacro:table prefix="table_" parent="rrbot_tool0">
+    <origin xyz="0 0 0" rpy="0 0 0"/>
+  </xacro:table>
 </robot>

File: ur3e_on_table/urdf/ur3e_on_table.urdf.xacro (robot description, xacro)
@@ -5,5 +5,5 @@
     <link name="world" />
     <xacro:table prefix="table_" parent="world">
-        <origin xyz="0 0 1" rpy="0 0 0" />
+        <origin xyz="0 0 0" rpy="0 0 0" />
     </xacro:table>
     <!-- robot name parameter -->
